File: connectors.kicad_sch (KiCad schematic)
At the start: 7 parts, among them J1 MicroFit_1x4, J2 MicroFit_1x4

Commit message: Updated from template, added graphics and JST-XH connectors
Parts:
- C8, C9: LCSC (none) -> C29936
- J1, J2: LCSC (none) -> C563846
Changed lines of the file:
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@@
 			)
 		)
-		(property "Description" "22U 25V X5R 0805"
+		(property "Description" "Unpolarized capacitor"
 			(at 114.3 52.07 0)
 			(effects
@@
 			)
 		)
-		(property "LCSC" ""
+		(property "LCSC" "C29936"
 			(at 114.3 52.07 0)
 			(effects
@@
 		)
 		(property "Manufacturer" "Samsung Electro-Mechanics"
+			(at 114.3 52.07 0)
+			(effects
+				(font
+					(size 1.27 1.27)
+				)
+				(hide yes)
+			)
+		)
+		(property "Sim.Pins" ""
 			(at 114.3 52.07 0)
 			(effects
@@
 			)
 		)
-		(property "Description" "Molex MicroFit3.0 1x4 Bus Connector"
+		(property "Description" "Generic connector, single row, 01x04, script generated"
 			(at 85.09 50.8 0)
 			(effects
@@
 		)
 		(property "Manufacturer" "Molex"
+			(at 85.09 50.8 0)
+			(effects
+				(font
+					(size 1.27 1.27)
+				)
+				(hide yes)
+			)
+		)
+		(property "LCSC" "C563846"
+			(at 85.09 50.8 0)
+			(effects
+				(font
+					(size 1.27 1.27)
+				)
+				(hide yes)
+			)
+		)
+		(property "Sim.Pins" ""
 			(at 85.09 50.8 0)
 			(effects
@@
 			)
 		)
-		(property "Description" "22U 25V X5R 0805"
+		(property "Description" "Unpolarized capacitor"
 			(at 121.92 52.07 0)
 			(effects
@@
 			)
 		)
-		(property "LCSC" ""
+		(property "LCSC" "C29936"
 			(at 121.92 52.07 0)
 			(effects
@@
 		)
 		(property "Manufacturer" "Samsung Electro-Mechanics"
+			(at 121.92 52.07 0)
+			(effects
+				(font
+					(size 1.27 1.27)
+				)
+				(hide yes)
+			)
+		)
+		(property "Sim.Pins" ""
 			(at 121.92 52.07 0)
 			(effects
@@
 		)
 		(property "Manufacturer" "Stackpole Electronics Inc"
+			(at 105.41 91.44 90)
+			(effects
+				(font
+					(size 1.27 1.27)
+				)
+				(hide yes)
+			)
+		)
+		(property "Sim.Pins" ""
 			(at 105.41 91.44 90)
 			(effects
@@
 			)
 		)
-		(property "Description" "Molex MicroFit3.0 1x4 Bus Connector"
+		(property "Description" "Generic connector, single row, 01x04, script generated"
 			(at 85.09 73.66 0)
 			(effects
@@
 		)
 		(property "Manufacturer" "Molex"
+			(at 85.09 73.66 0)
+			(effects
+				(font
+					(size 1.27 1.27)
+				)
+				(hide yes)
+			)
+		)
+		(property "LCSC" "C563846"
+			(at 85.09 73.66 0)
+			(effects
+				(font
+					(size 1.27 1.27)
+				)
+				(hide yes)
+			)
+		)
+		(property "Sim.Pins" ""
 			(at 85.09 73.66 0)
 			(effects
@@
 		)
 		(property "Manufacturer" "Keystone Electronics"
+			(at 104.14 55.88 0)
+			(effects
+				(font
+					(size 1.27 1.27)
+				)
+				(hide yes)
+			)
+		)
+		(property "Sim.Pins" ""
 			(at 104.14 55.88 0)
 			(effects
@@
 			(at 104.14 48.26 0)
 			(effects
+				(font
+					(size 1.27 1.27)
+				)
+				(hide yes)
+			)
+		)
+		(property "Sim.Pins" ""
+			(at 104.14 48.26 0)
+			(effects
