File: canbus.kicad_sch (KiCad schematic)
At the start: 12 parts, among them U1 MCP2562FD, U2 MCP2518FD, Y1 40 MHz

Commit message: Updated from template, added graphics and JST-XH connectors
Parts:
- C1, C2: LCSC (none) -> C1634
- C3, C5, C7: LCSC (none) -> C913912
- C4, C6: LCSC (none) -> C29936
- U1: LCSC (none) -> C511335; MPN MCP2562FDT-E/SN -> MCP2562FDT-H/SN; Manufacturer Microchip Technology -> Microchip
- U2: LCSC (none) -> C626758; Manufacturer Microchip Technology -> Microchip
- Y1: LCSC (none) -> C5357833
Changed lines of the file:
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@@
 			)
 		)
-		(property "Description" "10P 50V C0G 0603"
+		(property "Description" "Unpolarized capacitor"
 			(at 154.94 68.58 0)
 			(effects
@@
 		)
 		(property "Manufacturer" "Samsung Electro-Mechanics"
+			(at 154.94 68.58 0)
+			(effects
+				(font
+					(size 1.27 1.27)
+				)
+				(hide yes)
+			)
+		)
+		(property "LCSC" "C1634"
+			(at 154.94 68.58 0)
+			(effects
+				(font
+					(size 1.27 1.27)
+				)
+				(hide yes)
+			)
+		)
+		(property "Sim.Pins" ""
 			(at 154.94 68.58 0)
 			(effects
@@
 			)
 		)
+		(property "Sim.Pins" ""
+			(at 119.38 64.77 0)
+			(effects
+				(font
+					(size 1.27 1.27)
+				)
+				(hide yes)
+			)
+		)
 		(pin "1"
 		)
@@
 			)
 		)
-		(property "Description" "1U 25V X7R 0603"
+		(property "Description" "Unpolarized capacitor"
 			(at 99.06 48.26 0)
 			(effects
@@
 			)
 		)
-		(property "LCSC" ""
+		(property "LCSC" "C29936"
 			(at 99.06 48.26 0)
 			(effects
@@
 		)
 		(property "Manufacturer" "Samsung Electro-Mechanics"
+			(at 99.06 48.26 0)
+			(effects
+				(font
+					(size 1.27 1.27)
+				)
+				(hide yes)
+			)
+		)
+		(property "Sim.Pins" ""
 			(at 99.06 48.26 0)
 			(effects
@@
 			)
 		)
-		(property "Description" "0.1U 50V X7R 0603"
+		(property "Description" "Unpolarized capacitor"
 			(at 91.44 48.26 0)
 			(effects
@@
 			)
 		)
-		(property "LCSC" ""
+		(property "LCSC" "C913912"
 			(at 91.44 48.26 0)
 			(effects
@@
 		)
 		(property "Manufacturer" "Samsung Electro-Mechanics"
+			(at 91.44 48.26 0)
+			(effects
+				(font
+					(size 1.27 1.27)
+				)
+				(hide yes)
+			)
+		)
+		(property "Sim.Pins" ""
 			(at 91.44 48.26 0)
 			(effects
@@
 			)
 		)
+		(property "Sim.Pins" ""
+			(at 121.92 66.04 0)
+			(effects
+				(font
+					(size 1.27 1.27)
+				)
+				(hide yes)
+			)
+		)
 		(pin "1"
 		)
@@
 			)
 		)
-		(property "Description" "1U 25V X7R 0603"
+		(property "Description" "Unpolarized capacitor"
 			(at 80.01 48.26 0)
 			(effects
@@
 			)
 		)
-		(property "LCSC" ""
+		(property "LCSC" "C29936"
 			(at 80.01 48.26 0)
 			(effects
@@
 		)
 		(property "Manufacturer" "Samsung Electro-Mechanics"
+			(at 80.01 48.26 0)
+			(effects
+				(font
+					(size 1.27 1.27)
+				)
+				(hide yes)
+			)
+		)
+		(property "Sim.Pins" ""
 			(at 80.01 48.26 0)
 			(effects
@@
 			)
 		)
-		(property "Description" "0.1U 50V X7R 0603"
+		(property "Description" "Unpolarized capacitor"
 			(at 127 48.26 0)
 			(effects
@@
 			)
 		)
-		(property "LCSC" ""
+		(property "LCSC" "C913912"
 			(at 127 48.26 0)
 			(effects
@@
 		)
 		(property "Manufacturer" "Samsung Electro-Mechanics"
+			(at 127 48.26 0)
+			(effects
+				(font
+					(size 1.27 1.27)
+				)
+				(hide yes)
+			)
+		)
+		(property "Sim.Pins" ""
 			(at 127 48.26 0)
 			(effects
@@
 			)
 		)
-		(property "Description" "10P 50V C0G 0603"
+		(property "Description" "Unpolarized capacitor"
 			(at 140.97 68.58 0)
 			(effects
@@
 		)
 		(property "Manufacturer" "Samsung Electro-Mechanics"
+			(at 140.97 68.58 0)
+			(effects
+				(font
+					(size 1.27 1.27)
+				)
+				(hide yes)
+			)
+		)
+		(property "LCSC" "C1634"
+			(at 140.97 68.58 0)
+			(effects
+				(font
+					(size 1.27 1.27)
+				)
+				(hide yes)
+			)
+		)
+		(property "Sim.Pins" ""
 			(at 140.97 68.58 0)
 			(effects
@@
 			)
 		)
-		(property "MPN" "MCP2562FDT-E/SN"
+		(property "MPN" "MCP2562FDT-H/SN"
 			(at 107.95 67.31 0)
 			(effects
@@
 			)
 		)
-		(property "Manufacturer" "Microchip Technology"
+		(property "Manufacturer" "Microchip"
 			(at 107.95 67.31 0)
 			(effects
@@
 			)
 		)
-		(property "LCSC" ""
+		(property "LCSC" "C511335"
 			(at 107.95 67.31 0)
 			(effects
@@
 		)
 		(property "Digikey" "MCP2562FDT-E/SNCT-ND"
+			(at 107.95 67.31 0)
+			(effects
+				(font
+					(size 1.27 1.27)
+				)
+				(hide yes)
+			)
+		)
+		(property "Sim.Pins" ""
 			(at 107.95 67.31 0)
 			(effects
@@
 			)
 		)
-		(property "Manufacturer" "Microchip Technology"
+		(property "Manufacturer" "Microchip"
 			(at 66.04 71.12 0)
 			(effects
@@
 			)
 		)
-		(property "LCSC" ""
+		(property "LCSC" "C626758"
 			(at 66.04 71.12 0)
 			(effects
@@
 		)
 		(property "Digikey" "MCP2518FDT-E/SLCT-ND "
+			(at 66.04 71.12 0)
+			(effects
+				(font
+					(size 1.27 1.27)
+				)
+				(hide yes)
+			)
+		)
+		(property "Sim.Pins" ""
 			(at 66.04 71.12 0)
 			(effects
@@
 			)
 		)
-		(property "Description" "40 MHz ±10ppm Crystal 10pF 40 Ohms"
+		(property "Description" "Four pin crystal, GND on pins 2 and 4"
 			(at 148.59 64.77 0)
 			(effects
@@
 		)
 		(property "Manufacturer" "ECS Inc,"
+			(at 148.59 64.77 0)
+			(effects
+				(font
+					(size 1.27 1.27)
+				)
+				(hide yes)
+			)
+		)
+		(property "LCSC" "C5357833"
+			(at 148.59 64.77 0)
+			(effects
+				(font
+					(size 1.27 1.27)
+				)
+				(hide yes)
+			)
+		)
+		(property "Sim.Pins" ""
 			(at 148.59 64.77 0)
 			(effects
@@
 			)
 		)
-		(property "Description" "0.1U 50V X7R 0603"
+		(property "Description" "Unpolarized capacitor"
 			(at 72.39 48.26 0)
 			(effects
@@
 			)
 		)
-		(property "LCSC" ""
+		(property "LCSC" "C913912"
 			(at 72.39 48.26 0)
 			(effects
@@
 			(at 72.39 48.26 0)
 			(effects
+				(font
+					(size 1.27 1.27)
+				)
+				(hide yes)
+			)
+		)
+		(property "Sim.Pins" ""
+			(at 72.39 48.26 0)
+			(effects

Commit message: Add production date and up revision
Parts:
- C3, C5, C7: Digikey 490-5798-1-ND -> 1276-CL10B104KB8NNNLCT-ND
Changed lines of the file:
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@@
 			)
 		)
-		(property "Digikey" "490-5798-1-ND"
+		(property "Digikey" "1276-CL10B104KB8NNNLCT-ND"
 			(at 91.44 48.26 0)
 			(effects
@@
 			)
 		)
-		(property "Digikey" "490-5798-1-ND"
+		(property "Digikey" "1276-CL10B104KB8NNNLCT-ND"
 			(at 127 48.26 0)
 			(effects
@@
 			)
 		)
-		(property "Digikey" "490-5798-1-ND"
+		(property "Digikey" "1276-CL10B104KB8NNNLCT-ND"
 			(at 72.39 48.26 0)
 			(effects
