File: relays.kicad_sch (KiCad schematic)
At the start: 18 parts, among them J3 Screw_Terminal_01x08, K1 G6DN-1A DC5, K2 G6DN-1A DC5, K3 G6DN-1A DC5, K4 G6DN-1A DC5, Q1 Q_NMOS, Q2 Q_NMOS, Q3 Q_NMOS, Q4 Q_NMOS

Commit message: Add production date and up revision
Parts:
- C13, C14, C15, C16: Digikey 490-5798-1-ND -> 1276-CL10B104KB8NNNLCT-ND
Changed lines of the file:
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@@
 			)
 		)
-		(property "Digikey" "490-5798-1-ND"
+		(property "Digikey" "1276-CL10B104KB8NNNLCT-ND"
 			(at 68.58 91.44 90)
 			(effects
@@
 			)
 		)
-		(property "Digikey" "490-5798-1-ND"
+		(property "Digikey" "1276-CL10B104KB8NNNLCT-ND"
 			(at 68.58 69.85 90)
 			(effects
@@
 			)
 		)
-		(property "Digikey" "490-5798-1-ND"
+		(property "Digikey" "1276-CL10B104KB8NNNLCT-ND"
 			(at 68.58 31.75 90)
 			(effects
@@
 			)
 		)
-		(property "Digikey" "490-5798-1-ND"
+		(property "Digikey" "1276-CL10B104KB8NNNLCT-ND"
 			(at 68.58 49.53 90)
 			(effects
